File: Remote_PCB/ESP_board/ESP_board.kicad_pcb (KiCad board)
At the start: 2 copper layers, 12 parts, among them J1 leftside, J2 rightside, J3 Conn_01x03_Male, J4 breakout, J6 Batt_Input

Commit message: Finished Layout
Parts:
- moved R1 2.12 mm to (147.3, 106.8)
- moved R2 1.91 mm to (147.3, 113.8)
Connections:
- J4 pad 7: /4 -> /26
Routing:
- net +3V3: track 0.00 -> 53.9 mm
- net /21: track 0.00 -> 46.5 mm
- net /TX: track 0.00 -> 44.4 mm
- net /RX: track 0.00 -> 44.4 mm
- net /32: track 0.00 -> 17.8 mm
- net /26: track 0.00 -> 15.7 mm
- net /12: track 0.00 -> 14.7 mm
- net Net-(D2-Pad2): track 0.00 -> 7.14 mm
- net Net-(D1-Pad2): track 0.00 -> 7.14 mm
- net /16: track 43.4 -> 44.8 mm
- removed copper zone on F.Cu, net +3V3
Changed lines of the file:
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@@
-(kicad_pcb (version 20171130) (host pcbnew "(5.1.0)-1")
+(kicad_pcb (version 20171130) (host pcbnew "(5.1.2)-2")
   (general
     (thickness 1.6)
     (drawings 4)
-    (tracks 8)
+    (tracks 40)
     (zones 0)
     (modules 12)
@@
       (net 10 /32))
     (pad 7 thru_hole oval (at 0 15.24 90) (size 1.7 1.7) (drill 1) (layers *.Cu *.Mask)
-      (net 32 /4))
+      (net 13 /26))
     (pad 8 thru_hole oval (at 0 17.78 90) (size 1.7 1.7) (drill 1) (layers *.Cu *.Mask)
       (net 26 /21))
@@
   )
   (module Resistors_SMD:R_0603_HandSoldering (layer F.Cu)
-    (at 149.225 113.835 90)
+    (at 147.32 113.835 90)
     (descr "Resistor SMD 0603, hand soldering")
     (tags "resistor 0603")
@@
   )
   (module Resistors_SMD:R_0603_HandSoldering (layer F.Cu)
-    (at 149.225 107.78 90)
+    (at 147.32 106.85 90)
     (descr "Resistor SMD 0603, hand soldering")
     (tags "resistor 0603")
@@
   (gr_line (start 158.75 69.85) (end 158.75 120.65) (layer F.SilkS) (width 0.12))
   (gr_line (start 88.9 69.85) (end 158.75 69.85) (layer F.SilkS) (width 0.12))
+  (segment (start 151.765 107.95) (end 153.67 106.045) (width 0.25) (layer F.Cu) (net 2))
+  (segment (start 147.32 107.95) (end 151.765 107.95) (width 0.25) (layer F.Cu) (net 2))
+  (segment (start 151.765 114.935) (end 153.67 113.03) (width 0.25) (layer F.Cu) (net 3))
+  (segment (start 147.32 114.935) (end 151.765 114.935) (width 0.25) (layer F.Cu) (net 3))
+  (segment (start 116.205 110.585) (end 104.14 98.52) (width 0.25) (layer F.Cu) (net 4))
+  (segment (start 116.205 112.395) (end 116.205 110.585) (width 0.25) (layer F.Cu) (net 4))
+  (segment (start 94.445 79.375) (end 93.345 79.375) (width 0.25) (layer F.Cu) (net 4))
+  (segment (start 110.395001 99.084001) (end 110.395001 95.325001) (width 0.25) (layer F.Cu) (net 4))
+  (segment (start 109.784001 99.695001) (end 110.395001 99.084001) (width 0.25) (layer F.Cu) (net 4))
+  (segment (start 110.395001 95.325001) (end 94.445 79.375) (width 0.25) (layer F.Cu) (net 4))
+  (segment (start 104.215001 99.695001) (end 109.784001 99.695001) (width 0.25) (layer F.Cu) (net 4))
+  (segment (start 104.14 99.62) (end 104.215001 99.695001) (width 0.25) (layer F.Cu) (net 4))
+  (segment (start 104.14 98.52) (end 104.14 99.62) (width 0.25) (layer F.Cu) (net 4))
   (segment (start 94.547081 84.455) (end 93.345 84.455) (width 0.25) (layer F.Cu) (net 6))
   (segment (start 96.357081 84.455) (end 94.547081 84.455) (width 0.25) (layer F.Cu) (net 6))
   (segment (start 109.22 97.317919) (end 96.357081 84.455) (width 0.25) (layer F.Cu) (net 6))
   (segment (start 109.22 98.52) (end 109.22 97.317919) (width 0.25) (layer F.Cu) (net 6))
-  (segment (start 149.225 106.53) (end 152.4 103.355) (width 0.25) (layer F.Cu) (net 31))
-  (segment (start 149.225 106.68) (end 149.225 106.53) (width 0.25) (layer F.Cu) (net 31))
+  (segment (start 119.38 102.87) (end 119.38 98.52) (width 0.25) (layer F.Cu) (net 10))
+  (segment (start 128.905 112.395) (end 119.38 102.87) (width 0.25) (layer F.Cu) (net 10))
+  (segment (start 127 107.95) (end 127 98.52) (width 0.25) (layer F.Cu) (net 13))
+  (segment (start 131.445 112.395) (end 127 107.95) (width 0.25) (layer F.Cu) (net 13))
+  (segment (start 136.525 100.425) (end 134.62 98.52) (width 0.25) (layer F.Cu) (net 16))
+  (segment (start 136.525 112.395) (end 136.525 100.425) (width 0.25) (layer F.Cu) (net 16))
+  (segment (start 147.32 112.735) (end 147.32 112.585) (width 0.25) (layer F.Cu) (net 21))
+  (segment (start 112.609999 73.874999) (end 111.76 73.025) (width 0.25) (layer F.Cu) (net 24))
+  (segment (start 112.935001 74.200001) (end 112.609999 73.874999) (width 0.25) (layer F.Cu) (net 24))
+  (segment (start 112.935001 101.505001) (end 112.935001 74.200001) (width 0.25) (layer F.Cu) (net 24))
+  (segment (start 123.825 112.395) (end 112.935001 101.505001) (width 0.25) (layer F.Cu) (net 24))
+  (segment (start 115.149999 73.874999) (end 114.3 73.025) (width 0.25) (layer F.Cu) (net 25))
+  (segment (start 115.475001 74.200001) (end 115.149999 73.874999) (width 0.25) (layer F.Cu) (net 25))
+  (segment (start 115.475001 101.505001) (end 115.475001 74.200001) (width 0.25) (layer F.Cu) (net 25))
+  (segment (start 126.365 112.395) (end 115.475001 101.505001) (width 0.25) (layer F.Cu) (net 25))
+  (segment (start 117.689999 73.874999) (end 116.84 73.025) (width 0.25) (layer F.Cu) (net 26))
+  (segment (start 128.175001 84.360001) (end 117.689999 73.874999) (width 0.25) (layer F.Cu) (net 26))
+  (segment (start 128.175001 106.585001) (end 128.175001 84.360001) (width 0.25) (layer F.Cu) (net 26))
+  (segment (start 133.985 112.395) (end 128.175001 106.585001) (width 0.25) (layer F.Cu) (net 26))
   (segment (start 152.4 93.32) (end 132.08 73) (width 0.25) (layer F.Cu) (net 31))
   (segment (start 152.4 103.355) (end 152.4 93.32) (width 0.25) (layer F.Cu) (net 31))
+  (segment (start 150.005 105.75) (end 147.32 105.75) (width 0.25) (layer F.Cu) (net 31))
+  (segment (start 152.4 103.355) (end 150.005 105.75) (width 0.25) (layer F.Cu) (net 31))
   (zone (net 1) (net_name GND) (layer B.Cu) (hatch edge 0.508)
     (connect_pads (clearance 0.508))
@@
     (polygon
       (pts
-        (xy 158.75 120.65) (xy 88.9 120.65) (xy 88.9 69.85) (xy 158.75 69.85)
+        (xy 88.9 69.85) (xy 88.9 120.65) (xy 158.75 120.65) (xy 158.75 69.85)
       )
     )
-    (polygon
-      (pts
-        (xy 90.17 76.2) (xy 90.17 86.995) (xy 100.33 86.995) (xy 100.33 100.33) (xy 106.045 100.33)
-        (xy 106.045 76.2)
-      )
-    )
-  )
-  (zone (net 4) (net_name +3V3) (layer F.Cu) (hatch edge 0.508)
-    (connect_pads (clearance 0.508))
-    (min_thickness 0.254)
-    (fill yes (arc_segments 32) (thermal_gap 0.508) (thermal_bridge_width 0.508))
-    (polygon
-      (pts
-        (xy 100.965 99.695) (xy 100.965 80.645) (xy 90.805 80.645) (xy 90.805 76.835) (xy 105.41 76.835)
-        (xy 105.41 99.695)
-      )
-    )
