File: Remote_PCB/ESP_board/ESP_board.sch (KiCad schematic (older format))
At the start: 9 parts, among them J1 leftside, J2 rightside, J3 Conn_01x03_Male, J4 breakout, J6 Batt_Input

Commit message: Finished Layout
Connections:
- net 26: now also J4.7 (Pin_7)
- net 4: no longer J4.7 (Pin_7)
Changed lines of the file:
@@
 $EndComp
 Text Label 5200 5650 0    50   ~ 0
-4
+26
 Text Label 5200 5750 0    50   ~ 0
 21
